File: ArduinoISP.kicad_pcb (KiCad board)
At the start: 2 copper layers, 43.2 x 17.8 mm, 15 parts, among them J1 Analog, J2 Digital, J3 AVR-ISP-10, J4 AVR-ISP-6

Commit message: try double ended
Parts:
- added J5: ISP-6-Socket, ArduinoISP:IDC-Header_2x03_P2.54mm_Horizontal, B.Cu at (141.4, 88.6)
- J3: value AVR-ISP-10 -> ISP-10
- J4: value AVR-ISP-6 -> ISP-6-Pins
- moved J4 40.3 mm to (101.7, 93.7), turned to 180 degrees
- moved D1 27.5 mm to (133.8, 88.8)
- moved R1 27.5 mm to (130.0, 88.8)
- moved D2 27.4 mm to (133.8, 91.1)
- moved R2 27.4 mm to (130.0, 91.1)
- moved D3 27.4 mm to (133.8, 93.4)
- moved R3 27.4 mm to (130.0, 93.4)
- moved JP1 26.9 mm to (108.5, 88.6)
Routing:
- net GND: track 79.6 -> 0.00 mm, vias 1 -> 0
- net /D12/MISO: track 45.1 -> 0.00 mm, vias 2 -> 0
- net /D13/SCK: track 44.8 -> 0.00 mm
- net /*D10/SS: track 43.3 -> 0.00 mm
- net /*D11/MOSI: track 43.1 -> 0.00 mm, vias 1 -> 0
- net +3V3: track 31.3 -> 0.00 mm
- net Net-(J3-VCC): track 28.9 -> 0.00 mm
- net /D7: track 14.5 -> 0.00 mm
- net +5V: track 13.3 -> 0.00 mm, vias 1 -> 0
- net /D8: track 11.5 -> 0.00 mm
- net /*D9: track 9.07 -> 0.00 mm
- net Net-(D3-K): track 2.02 -> 0.00 mm
- net Net-(D2-K): track 2.02 -> 0.00 mm
- net Net-(D1-K): track 2.02 -> 0.00 mm

Commit message: redo board
Routing:
- net GND: track 0.00 -> 85.1 mm, vias 0 -> 11
- net /*D10/SS: track 0.00 -> 60.2 mm, vias 0 -> 1
- net /D13/SCK: track 0.00 -> 54.6 mm
- net /D12/MISO: track 0.00 -> 50.2 mm, vias 0 -> 2
- net /*D11/MOSI: track 0.00 -> 50.0 mm, vias 0 -> 1
- net Net-(J3-VCC): track 0.00 -> 46.6 mm, vias 0 -> 1
- net +5V: track 0.00 -> 31.2 mm
- net /D7: track 0.00 -> 28.2 mm
- net /D8: track 0.00 -> 27.1 mm
- net /*D9: track 0.00 -> 25.5 mm
- net +3V3: track 0.00 -> 5.97 mm
- net Net-(D3-K): track 0.00 -> 2.02 mm
- net Net-(D2-K): track 0.00 -> 2.02 mm
- net Net-(D1-K): track 0.00 -> 2.02 mm
Other:
- board text added: "Arduino as ISP"

Commit message: part numbers
Changed lines of the file:
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@@
 			)
 		)
+		(property "MPN" "2541FV-15P-B"
+			(at 0 0 90)
+			(unlocked yes)
+			(layer "F.Fab")
+			(hide yes)
+			(effects
+				(font
+					(size 1 1)
+					(thickness 0.15)
+				)
+			)
+		)
 		(property ki_fp_filters "Connector*:*_1x??_*")
 		(sheetname "/")
@@
 			)
 		)
+		(property "MPN" "2541FV-15P-B"
+			(at 0 0 90)
+			(unlocked yes)
+			(layer "F.Fab")
+			(hide yes)
+			(effects
+				(font
+					(size 1 1)
+					(thickness 0.15)
+				)
+			)
+		)
 		(property ki_fp_filters "Connector*:*_1x??_*")
 		(sheetname "/")
@@
 			)
 		)
+		(property "MPN" "FRC0603F2200TS"
+			(at 0 0 180)
+			(unlocked yes)
+			(layer "F.Fab")
+			(hide yes)
+			(effects
+				(font
+					(size 1 1)
+					(thickness 0.15)
+				)
+			)
+		)
 		(property ki_fp_filters "R_*")
 		(sheetname "/")
@@
 			)
 		)
+		(property "MPN" "GL0603UY01"
+			(at 0 0 0)
+			(unlocked yes)
+			(layer "F.Fab")
+			(hide yes)
+			(effects
+				(font
+					(size 1 1)
+					(thickness 0.15)
+				)
+			)
+		)
 		(property ki_fp_filters "LED* LED_SMD:* LED_THT:*")
 		(sheetname "/")
@@
 			)
 		)
+		(property "MPN" "DS1013-06SSiB1-B-0"
+			(at 0 0 180)
+			(unlocked yes)
+			(layer "F.Fab")
+			(hide yes)
+			(effects
+				(font
+					(size 1 1)
+					(thickness 0.15)
+				)
+			)
+		)
 		(property ki_fp_filters "IDC?Header*2x03* Pin?Header*2x03*")
 		(sheetname "/")
@@
 			)
 		)
+		(property "MPN" "FRC0603F2200TS"
+			(at 0 0 180)
+			(unlocked yes)
+			(layer "F.Fab")
+			(hide yes)
+			(effects
+				(font
+					(size 1 1)
+					(thickness 0.15)
+				)
+			)
+		)
 		(property ki_fp_filters "R_*")
 		(sheetname "/")
@@
 			)
 		)
+		(property "MPN" "FRC0603F2200TS"
+			(at 0 0 180)
+			(unlocked yes)
+			(layer "F.Fab")
+			(hide yes)
+			(effects
+				(font
+					(size 1 1)
+					(thickness 0.15)
+				)
+			)
+		)
 		(property ki_fp_filters "R_*")
 		(sheetname "/")
@@
 			)
 		)
+		(property "MPN" "GL0603UR01"
+			(at 0 0 0)
+			(unlocked yes)
+			(layer "F.Fab")
+			(hide yes)
+			(effects
+				(font
+					(size 1 1)
+					(thickness 0.15)
+				)
+			)
+		)
 		(property ki_fp_filters "LED* LED_SMD:* LED_THT:*")
 		(sheetname "/")
@@
 			)
 		)
+		(property "MPN" "GL0603UG01"
+			(at 0 0 0)
+			(unlocked yes)
+			(layer "F.Fab")
+			(hide yes)
+			(effects
+				(font
+					(size 1 1)
+					(thickness 0.15)
+				)
+			)
+		)
 		(property ki_fp_filters "LED* LED_SMD:* LED_THT:*")
 		(sheetname "/")
@@
 			)
 		)
+		(property "MPN" "DS1013-10SSiB1-B-0"
+			(at 0 0 270)
+			(unlocked yes)
+			(layer "B.Fab")
+			(hide yes)
+			(effects
+				(font
+					(size 1 1)
+					(thickness 0.15)
+				)
+				(justify mirror)
+			)
+		)
 		(property ki_fp_filters "IDC?Header*2x05* Pin?Header*2x05*")
 		(sheetname "/")
@@
 			)
 		)
+		(property "MPN" "DS1023-32-2x3V8"
+			(at 0 0 180)
+			(unlocked yes)
+			(layer "B.Fab")
+			(hide yes)
+			(effects
+				(font
+					(size 1 1)
+					(thickness 0.15)
+				)
+				(justify mirror)
+			)
+		)
 		(property ki_fp_filters "IDC?Header*2x03* Pin?Header*2x03*")
 		(sheetname "/")
@@
 			)
 		)
+		(property "MPN" "2541WV-03P"
+			(at 0 0 180)
+			(unlocked yes)
+			(layer "B.Fab")
+			(hide yes)
+			(effects
+				(font
+					(size 1 1)
+					(thickness 0.15)
+				)
+				(justify mirror)
+			)
+		)
+		(property "MPN2" "M254D-02-065-B"
+			(at 0 0 180)
+			(unlocked yes)
+			(layer "B.Fab")
+			(hide yes)
+			(effects
+				(font
+					(size 1 1)
+					(thickness 0.15)
+				)
+				(justify mirror)
+			)
+		)
 		(property ki_fp_filters "Jumper* TestPoint*3Pads* TestPoint*Bridge*")
 		(sheetname "/")
@@
 	)
 	(segment
-		(start 136.334 90.168391)
-		(end 136.322 90.180391)
+		(start 136.449 87.427)
+		(end 136.449 91.5945)
 		(width 0.25)
 		(layer "F.Cu")
@@
 	)
 	(segment
-		(start 116.51 83.49)
-		(end 118.772 85.752)
-		(width 0.25)
-		(layer "F.Cu")
-		(net "/D7")
-	)
-	(segment
-		(start 136.322 88.088609)
-		(end 136.334 88.100608)
+		(start 134.774 85.752)
+		(end 136.449 87.427)
 		(width 0.25)
 		(layer "F.Cu")
@@
 	)
 	(segment
-		(start 136.322 87.3)
-		(end 136.322 88.088609)
-		(width 0.25)
-		(layer "F.Cu")
-		(net "/D7")
-	)
-	(segment
-		(start 136.322 90.180391)
-		(end 136.322 91.7215)
-		(width 0.25)
-		(layer "F.Cu")
-		(net "/D7")
-	)
-	(segment
-		(start 136.334 88.100608)
-		(end 136.334 90.168391)
-		(width 0.25)
-		(layer "F.Cu")
-		(net "/D7")
-	)
-	(segment
-		(start 136.322 91.7215)
+		(start 136.449 91.5945)
 		(end 134.6475 93.396)
 		(width 0.25)
@@
 	)
 	(segment
-		(start 134.774 85.752)
-		(end 136.322 87.3)
+		(start 116.51 83.49)
+		(end 118.772 85.752)
 		(width 0.25)
 		(layer "F.Cu")
