File: ArduinoISP.kicad_sch (KiCad schematic)
At the start: 11 parts, among them J1 Analog, J2 Digital, J3 AVR-ISP-10, J4 AVR-ISP-6

Commit message: try double ended
Parts:
- added J5: ISP-6-Socket, ArduinoISP:IDC-Header_2x03_P2.54mm_Horizontal, symbol Connector:AVR-ISP-6
- J3: value AVR-ISP-10 -> ISP-10
- J4: value AVR-ISP-6 -> ISP-6-Pins
Connections:
- net *D10/SS: now also J5.5 (~{RST})
- net *D11/MOSI: now also J5.4 (MOSI)
- net D12/MISO: now also J5.1 (MISO)
- net D13/SCK: now also J5.3 (SCK)
- net GND: now also J5.6 (GND)
- net at J3.2 (VCC), J4.2 (VCC), JP1.2 (C): now also J5.2 (VCC)
Other:
- moved on the sheet: J4
Changed lines of the file:
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@@
+	)
+	(junction
+		(at 142.24 53.34)
+		(diameter 0)
+		(color 0 0 0 0)
 	)
 	(junction
@@
 		(color 0 0 0 0)
 	)
+	(junction
+		(at 142.24 30.48)
+		(diameter 0)
+		(color 0 0 0 0)
+	)
 	(no_connect
 		(at 17.78 57.15)
@@
 	(wire
 		(pts
-			(xy 101.6 53.34) (xy 152.4 53.34)
+			(xy 101.6 53.34) (xy 142.24 53.34)
 		)
 		(stroke
@@
 	(wire
 		(pts
+			(xy 142.24 53.34) (xy 181.61 53.34)
+		)
+		(stroke
+			(width 0)
+			(type default)
+		)
+	)
+	(wire
+		(pts
 			(xy 17.78 34.29) (xy 35.56 34.29)
 		)
@@
 	(wire
 		(pts
+			(xy 142.24 30.48) (xy 181.61 30.48)
+		)
+		(stroke
+			(width 0)
+			(type default)
+		)
+	)
+	(wire
+		(pts
 			(xy 55.88 34.29) (xy 71.12 34.29)
 		)
@@
 	(wire
 		(pts
-			(xy 101.6 30.48) (xy 152.4 30.48)
+			(xy 101.6 30.48) (xy 142.24 30.48)
 		)
 		(stroke
@@
 		)
 	)
+	(label "*D10{slash}SS"
+		(at 168.91 45.72 180)
+		(effects
+			(font
+				(size 1.27 1.27)
+			)
+			(justify right bottom)
+		)
+	)
 	(label "D8"
 		(at 88.9 85.09 180)
@@
 	)
 	(label "D12{slash}MISO"
+		(at 168.91 38.1 180)
+		(effects
+			(font
+				(size 1.27 1.27)
+			)
+			(justify right bottom)
+		)
+	)
+	(label "D12{slash}MISO"
 		(at 88.9 38.1 180)
+		(effects
+			(font
+				(size 1.27 1.27)
+			)
+			(justify right bottom)
+		)
+	)
+	(label "*D11{slash}MOSI"
+		(at 168.91 40.64 180)
 		(effects
 			(font
@@
 	)
 	(label "D12{slash}MISO"
-		(at 139.7 38.1 180)
+		(at 129.54 38.1 180)
 		(effects
 			(font
@@
 	)
 	(label "*D10{slash}SS"
-		(at 139.7 45.72 180)
+		(at 129.54 45.72 180)
 		(effects
 			(font
@@
 	)
 	(label "D13{slash}SCK"
-		(at 139.7 43.18 180)
+		(at 129.54 43.18 180)
+		(effects
+			(font
+				(size 1.27 1.27)
+			)
+			(justify right bottom)
+		)
+	)
+	(label "D13{slash}SCK"
+		(at 168.91 43.18 180)
 		(effects
 			(font
@@
 	)
 	(label "*D11{slash}MOSI"
-		(at 139.7 40.64 180)
+		(at 129.54 40.64 180)
 		(effects
 			(font
@@
 				(path "/0d35483a-0b12-46cc-b9f2-896fd6831779"
 					(reference "#FLG03")
+					(unit 1)
+				)
+			)
+		)
+	)
+	(symbol
+		(lib_id "Connector:AVR-ISP-6")
+		(at 179.07 43.18 0)
+		(mirror y)
+		(unit 1)
+		(body_style 1)
+		(exclude_from_sim no)
+		(in_bom yes)
+		(on_board yes)
+		(in_pos_files yes)
+		(dnp no)
+		(fields_autoplaced yes)
+		(property "Reference" "J5"
+			(at 187.96 40.6399 0)
+			(show_name no)
+			(do_not_autoplace no)
+			(effects
+				(font
+					(size 1.27 1.27)
+				)
+				(justify right)
+			)
+		)
+		(property "Value" "ISP-6-Socket"
+			(at 187.96 43.1799 0)
+			(show_name no)
+			(do_not_autoplace no)
+			(effects
+				(font
+					(size 1.27 1.27)
+				)
+				(justify right)
+			)
+		)
+		(property "Footprint" "ArduinoISP:IDC-Header_2x03_P2.54mm_Horizontal"
+			(at 185.42 41.91 90)
+			(hide yes)
+			(show_name no)
+			(do_not_autoplace no)
+			(effects
+				(font
+					(size 1.27 1.27)
+				)
+			)
+		)
+		(property "Datasheet" ""
+			(at 211.455 57.15 0)
+			(hide yes)
+			(show_name no)
+			(do_not_autoplace no)
+			(effects
+				(font
+					(size 1.27 1.27)
+				)
+			)
+		)
+		(property "Description" "Atmel 6-pin ISP connector"
+			(at 179.07 43.18 0)
+			(hide yes)
+			(show_name no)
+			(do_not_autoplace no)
+			(effects
+				(font
+					(size 1.27 1.27)
+				)
+			)
+		)
+		(pin "4"
+		)
+		(pin "3"
+		)
+		(pin "2"
+		)
+		(pin "1"
+		)
+		(pin "6"
+		)
+		(pin "5"
+		)
+		(instances
+			(project "ArduinoISP"
+				(path "/0d35483a-0b12-46cc-b9f2-896fd6831779"
+					(reference "J5")
 					(unit 1)
 				)
@@
 			)
 		)
-		(property "Value" "AVR-ISP-10"
+		(property "Value" "ISP-10"
 			(at 107.95 43.1799 0)
 			(show_name no)
@@
 	(symbol
 		(lib_id "Connector:AVR-ISP-6")
-		(at 149.86 43.18 0)
+		(at 139.7 43.18 0)
 		(mirror y)
 		(unit 1)
@@
 		(fields_autoplaced yes)
 		(property "Reference" "J4"
-			(at 158.75 40.6399 0)
+			(at 148.59 40.6399 0)
 			(show_name no)
 			(do_not_autoplace no)
@@
 			)
 		)
-		(property "Value" "AVR-ISP-6"
-			(at 158.75 43.1799 0)
+		(property "Value" "ISP-6-Pins"
+			(at 148.59 43.1799 0)
 			(show_name no)
 			(do_not_autoplace no)
@@
 		)
 		(property "Footprint" "ArduinoISP:IDC-Header_2x03_P2.54mm_Horizontal"
-			(at 156.21 41.91 90)
+			(at 146.05 41.91 90)
 			(hide yes)
 			(show_name no)
@@
 		)
 		(property "Datasheet" ""
-			(at 182.245 57.15 0)
+			(at 172.085 57.15 0)
 			(hide yes)
 			(show_name no)
@@
 		)
 		(property "Description" "Atmel 6-pin ISP connector"
-			(at 149.86 43.18 0)
-			(hide yes)
-			(show_name no)
+			(at 139.7 43.18 0)
+			(hide yes)
+			(show_name no)

Commit message: part numbers
Parts:
- D1: MPN (none) -> GL0603UG01
- D2: MPN (none) -> GL0603UR01
- D3: MPN (none) -> GL0603UY01
- J1, J2: MPN (none) -> 2541FV-15P-B
- J3: MPN (none) -> DS1013-10SSiB1-B-0
- J4: MPN (none) -> DS1013-06SSiB1-B-0
- J5: MPN (none) -> DS1023-32-2x3V8
- JP1: MPN (none) -> 2541WV-03P; MPN2 (none) -> M254D-02-065-B; private KLC_S3.3 -> KLC_S5.1
- R1, R2, R3: MPN (none) -> FRC0603F2200TS
Changed lines of the file:
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@@
+			)
+		)
+		(property "MPN" "2541FV-15P-B"
+			(at 40.64 44.45 0)
+			(hide yes)
+			(show_name no)
+			(do_not_autoplace no)
+			(effects
+				(font
+					(size 1.27 1.27)
+				)
 			)
 		)
@@
 			)
 		)
+		(property "MPN" "2541FV-15P-B"
+			(at 50.8 44.45 0)
+			(hide yes)
+			(show_name no)
+			(do_not_autoplace no)
+			(effects
+				(font
+					(size 1.27 1.27)
+				)
+			)
+		)
 		(pin "1"
 		)
@@
 			)
 		)
+		(property "MPN" "DS1023-32-2x3V8"
+			(at 179.07 43.18 0)
+			(hide yes)
+			(show_name no)
+			(do_not_autoplace no)
+			(effects
+				(font
+					(size 1.27 1.27)
+				)
+			)
+		)
 		(pin "4"
 		)
@@
 			)
 		)
+		(property "MPN" "DS1013-10SSiB1-B-0"
+			(at 99.06 43.18 0)
+			(hide yes)
+			(show_name no)
+			(do_not_autoplace no)
+			(effects
+				(font
+					(size 1.27 1.27)
+				)
+			)
+		)
 		(pin "5"
 		)
@@
 			)
 		)
-		(property private "KLC_S3.3" "Graphical-Symbol: thickness is 6mm, fill is background"
-			(at 100.33 46.99 0)
-			(hide yes)
-			(show_name yes)
+		(property "MPN" "2541WV-03P"
+			(at 101.6 26.67 0)
+			(hide yes)
+			(show_name no)
+			(do_not_autoplace no)
+			(effects
+				(font
+					(size 1.27 1.27)
+				)
+			)
+		)
+		(property "MPN2" "M254D-02-065-B"
+			(at 101.6 26.67 0)
+			(hide yes)
+			(show_name no)
 			(do_not_autoplace no)
 			(effects
@@
 			)
 		)
+		(property "MPN" "FRC0603F2200TS"
+			(at 107.95 85.09 90)
+			(hide yes)
+			(show_name no)
+			(do_not_autoplace no)
+			(effects
+				(font
+					(size 1.27 1.27)
+				)
+			)
+		)
 		(pin "2"
 		)
@@
 			)
 		)
+		(property "MPN" "GL0603UY01"
+			(at 92.71 95.25 0)
+			(hide yes)
+			(show_name no)
+			(do_not_autoplace no)
+			(effects
+				(font
+					(size 1.27 1.27)
+				)
+			)
+		)
 		(pin "1"
 		)
@@
 			)
 		)
+		(property "MPN" "DS1013-06SSiB1-B-0"
+			(at 139.7 43.18 0)
+			(hide yes)
+			(show_name no)
+			(do_not_autoplace no)
+			(effects
+				(font
+					(size 1.27 1.27)
+				)
+			)
+		)
 		(pin "4"
 		)
@@
 			)
 		)
+		(property "MPN" "FRC0603F2200TS"
+			(at 107.95 95.25 90)
+			(hide yes)
+			(show_name no)
+			(do_not_autoplace no)
+			(effects
+				(font
+					(size 1.27 1.27)
+				)
+			)
+		)
 		(pin "2"
 		)
@@
 			)
 		)
+		(property "MPN" "GL0603UR01"
+			(at 92.71 85.09 0)
+			(hide yes)
+			(show_name no)
+			(do_not_autoplace no)
+			(effects
+				(font
+					(size 1.27 1.27)
+				)
+			)
+		)
 		(pin "1"
 		)
@@
 			)
 		)
+		(property "MPN" "FRC0603F2200TS"
+			(at 107.95 74.93 90)
+			(hide yes)
+			(show_name no)
+			(do_not_autoplace no)
+			(effects
+				(font
+					(size 1.27 1.27)
+				)
+			)
+		)
 		(pin "2"
 		)
@@
 			(at 92.71 74.93 0)
 			(hide yes)
+			(show_name no)
+			(do_not_autoplace no)
+			(effects
+				(font
+					(size 1.27 1.27)
+				)
+			)
+		)
+		(property "MPN" "GL0603UG01"
+			(at 92.71 74.93 0)
+			(hide yes)
